File: accel-mma84/accel-mma84.sch (KiCad schematic (older format))
At the start: 10 parts, among them IC1 AT24CS01-STUM, J2 CONN_01X10, J3 CONN_01X02, U1 MMA8452Q

Commit message: Adds a bridge for disabling write protection.
Parts:
- added P1: CONN_01X02, Socket_Strips:Socket_Strip_Straight_1x02, symbol CONN_01X02
- added R4: R, Resistors_SMD:R_0603, symbol R
Connections:
- net VCC: now also R4.1; no longer IC1.5 (WP)
- new net: IC1.5 (WP), P1.1 (P1)
- new net: P1.2 (P2), R4.2
Changed lines of the file:
@@
 EESchema Schematic File Version 2
+LIBS:freescale-ic
 LIBS:power
 LIBS:device
@@
 LIBS:contrib
 LIBS:valves
-LIBS:freescale-ic
+LIBS:accel-mma84-cache
 EELAYER 25 0
 EELAYER END
@@
 $EndComp
 Wire Wire Line
-	2250 5400 2100 5400
-Wire Wire Line
-	2100 5400 2100 4650
-Wire Wire Line
 	2650 4850 2650 4750
 Wire Wire Line
@@
 Wire Wire Line
 	3350 5250 3050 5250
+$Comp
+L CONN_01X02 P1
+U 1 1 55A36C14
+P 1650 5350
+F 0 "P1" H 1650 5500 50  0000 C CNN
+F 1 "CONN_01X02" V 1750 5350 50  0000 C CNN
+F 2 "Socket_Strips:Socket_Strip_Straight_1x02" H 1650 5350 60  0001 C CNN
+F 3 "" H 1650 5350 60  0000 C CNN
+	1    1650 5350
+	-1   0    0    1
+$EndComp
+$Comp
+L R R4
+U 1 1 55A36C59
+P 2100 5000
+F 0 "R4" V 2180 5000 50  0000 C CNN
+F 1 "R" V 2100 5000 50  0000 C CNN
+F 2 "Resistors_SMD:R_0603" V 2030 5000 30  0001 C CNN
+F 3 "" H 2100 5000 30  0000 C CNN
+	1    2100 5000
+	1    0    0    -1
+$EndComp
+Wire Wire Line
+	1850 5400 2250 5400
+Wire Wire Line
+	1850 5300 2100 5300
+Wire Wire Line
+	2100 5300 2100 5150
+Wire Wire Line
+	2100 4650 2100 4850
 $EndSCHEMATC
